Commit message: Add rack hip-height trials and T3 lift viewer updates

File: robot_demo_outputs/t3_robot/T3.urdf (robot description, URDF)
Before this commit: robot T3, 35 links, 34 joints
Links:
- removed link waist_connector_link
- added link telescopic_lift_base_link; collision box size=0.10 0.10 0.60; collision box size=0.16 0.16 0.02
- added link telescopic_lift_carriage_link; collision box size=0.08 0.08 0.55; visual box size=0.07 0.07 0.55
Joints:
- removed joint base_to_waist_connector
- removed joint waist_connector_to_waist_yaw
- added joint base_to_telescopic_lift: type fixed, parent base_link, child telescopic_lift_base_link, origin xyz=0 0 0 rpy=0 0 0
- added joint telescopic_lift_joint: type prismatic, parent telescopic_lift_base_link, child telescopic_lift_carriage_link, origin xyz=0 0 0.795 rpy=0 0 0, axis 0 0 1, limit lower=0 upper=0.55 effort=1000 velocity=0.25
- added joint telescopic_lift_to_waist_yaw: type fixed, parent telescopic_lift_carriage_link, child waist_yaw_link, origin xyz=0 0 0 rpy=0 0 0
